Commit message: Update arm_camera.xacro

File: arm_camera.xacro (robot description, xacro)
@@ -0,0 +1,25 @@
+<robot xmlns:xacro="http://www.ros.org/wiki/xacro">
+  <link name="camera_link">
+    <visual>
+      <geometry>
+        <box size="0.05 0.05 0.05"/>
+      </geometry>
+    </visual>
+  </link>
+  <joint name="camera_joint" type="fixed">
+    <parent link="base_link"/>
+    <child link="camera_link"/>
+  </joint>
+  <gazebo>
+    <sensor type="camera" name="camera">
+      <camera>
+        <horizontal_fov>1.047</horizontal_fov>
+        <image>
+          <width>800</width>
+          <height>600</height>
+        </image>
+      </camera>
+      <plugin name="gazebo_ros_camera" filename="libgazebo_ros_camera.so"/>
+    </sensor>
+  </gazebo>
+</robot>
